File: picise.kicad_sch (KiCad schematic)
At the start: 23 parts, among them J2 ANT_SMA, J4 TSM-103-01-L-SV, U1 CAT24C256, U2 MAX-M10S

Commit message: Update picise.kicad_sch
Parts:
- removed D1: SML522BUNWT86, LED_SMD_Rohm:SML522BUNWT86, symbol LED_SMD_Rohm:SML522BUNWT86
- removed SW?: ANT_ACTIVE, symbol Switch:SW_SPST
- added C10, C11, C2, C5, C6: 10uF, Capacitor_SMD:C_0603_1608Metric, symbol Device:C_Small
- added C12, C3, C7: 1uF, Capacitor_SMD:C_0603_1608Metric, symbol Device:C_Small
- added C13, C4, C8: 0.1uF, Capacitor_SMD:C_0603_1608Metric, symbol Device:C_Small
- added C?: 22pF, Capacitor_SMD:C_0603_1608Metric, symbol Device:C_Small
- added D1, D10, D11, D12, D13, D14, D15, D16, D17, D18, D19, D2, D20, D21, D22, D23, D24, D26, D27, D28, D29, D3, D30, D31, D32, D33, D34, D35, D36, D37, D38, D39, D4, D40, D41, D43, D44, D45, D46, D47, D48, D49, D5, D50, D51, D52, D53, D54, D55, D56, D57, D58, D59, D6, D60, D61, D62, D63, D64, D65, D66, D67, D68, D7, D8, D9: Green, Diode_SMD:D_0603_1608Metric, symbol Device:LED_Small_Filled
- added D42: Red, Diode_SMD:D_0603_1608Metric, symbol Device:LED_Small_Filled
- added D69: Blue, Diode_SMD:D_0603_1608Metric, symbol Device:LED_Small_Filled
- added JP1: ACT_PSV, symbol Jumper:Jumper_2_Bridged
- added R13, R14, R3, R4, R5: 20k, Resistor_SMD:R_0603_1608Metric, symbol Device:R_Small
- added R2: DNP, Resistor_SMD:R_0805_2012Metric_Pad1.20x1.40mm_HandSolder, symbol Device:R_Small
- added U2: PCA9557PW, Package_SO:TSSOP-16_4.4x5mm_P0.65mm, symbol Interface_Expansion:PCA9557PW
- added U4: IS31FL3731-QF, Package_DFN_QFN:QFN-28-1EP_4x4mm_P0.4mm_EP2.3x2.3mm, symbol Driver_LED:IS31FL3731-QF
- BT1: Digikey (none) -> MS621FE-FL11E
- C1: renamed from C?; footprint (none) -> Capacitor_SMD:C_0603_1608Metric; JLCPCB (none) -> C1671; MPN (none) -> CL10C470JB8NNNC; Manufacturer (none) -> Samsung
- C14: renamed from C2; footprint Capacitor_SMD:C_0805_2012Metric_Pad1.18x1.45mm_HandSolder -> Capacitor_SMD:C_0603_1608Metric; JLCPCB (none) -> C15849; MPN C0805C105J4RAC7800 -> CL10A105KB8NNNC; Manufacturer KEMET -> Samsung
- C9: renamed from C1; value 100n -> 0.1uF; footprint Capacitor_SMD:C_0805_2012Metric_Pad1.18x1.45mm_HandSolder -> Capacitor_SMD:C_0603_1608Metric; JLCPCB (none) -> C14663; MPN C0805C104J5RAC7800 -> CC0603KRX7R9BB104; Manufacturer KEMET -> Yageo
- D25: renamed from D2; footprint Diode_SMD:D_0805_2012Metric -> Diode_SMD:D_0603_1608Metric; JLCPCB (none) -> C143772; MPN SD0805S040S0R5 -> SD0603S040S0R2
- J1: renamed from J2; Digikey (none) -> SMA-J-P-H-ST-EM1
- J2: renamed from J?; Digikey (none) -> SSQ-120-03-G-D; MPN SSW-120-22-G-D-RA -> SSQ-120-03-G-D; PARTREV R -> (none); STANDARD Manufacturer Recommendations -> (none)
- J3: renamed from J4; Digikey (none) -> TSM-102-01-L-SV
- L1: renamed from L?; footprint (none) -> Inductor_SMD:L_0603_1608Metric; JLCPCB (none) -> C98076; MPN (none) -> LQW18AN47NG00D; Manufacturer (none) -> Murata
- R1: renamed from R?; footprint (none) -> Resistor_SMD:R_0603_1608Metric; JLCPCB (none) -> C22859; MPN (none) -> 0603WAF100JT5E; Manufacturer (none) -> uniroyal
- R10: renamed from R3; footprint Resistor_SMD:R_0805_2012Metric_Pad1.20x1.40mm_HandSolder -> Resistor_SMD:R_0603_1608Metric; JLCPCB (none) -> C23220; MPN RK73H2ATTD6200F -> 0603WAF6200T5E; Manufacturer KOA Speer -> uniroyal
- R11: renamed from R4; footprint Resistor_SMD:R_0805_2012Metric_Pad1.20x1.40mm_HandSolder -> Resistor_SMD:R_0603_1608Metric; JLCPCB (none) -> C4190; MPN RK73H2ATTD2201F -> 0603WAF2201T5E; Manufacturer KOA Speer -> uniroyal
- R12: renamed from R5; footprint Resistor_SMD:R_0805_2012Metric_Pad1.20x1.40mm_HandSolder -> Resistor_SMD:R_0603_1608Metric; JLCPCB (none) -> C4190; MPN RK73H2ATTD2201F -> 0603WAF2201T5E; Manufacturer KOA Speer -> uniroyal
- R6: renamed from R1; footprint Resistor_SMD:R_0805_2012Metric_Pad1.20x1.40mm_HandSolder -> Resistor_SMD:R_0603_1608Metric; JLCPCB (none) -> C23018; MPN RK73H2ARTTD3901F -> 0603WAF3901T5E; Manufacturer KOA Speer -> uniroyal
- R7: renamed from R2; footprint Resistor_SMD:R_0805_2012Metric_Pad1.20x1.40mm_HandSolder -> Resistor_SMD:R_0603_1608Metric; JLCPCB (none) -> C23018; MPN RK73H2ARTTD3901F -> 0603WAF3901T5E; Manufacturer KOA Speer -> uniroyal
- R8: renamed from R6; footprint Resistor_SMD:R_0805_2012Metric_Pad1.20x1.40mm_HandSolder -> Resistor_SMD:R_0603_1608Metric; JLCPCB (none) -> C23138; MPN RK73H2ATTD2800F -> 0603WAF3300T5E; Manufacturer KOA Speer -> uniroyal
- R9: renamed from R7; footprint Resistor_SMD:R_0805_2012Metric_Pad1.20x1.40mm_HandSolder -> Resistor_SMD:R_0603_1608Metric; JLCPCB (none) -> C23115; MPN RK73H2ARTTD80R6F -> 0603WAF806JT5E; Manufacturer KOA Speer -> uniroyal
- U3: renamed from U1; JLCPCB (none) -> C79987
- renumbered JP1 to JP2, JP2 to JP3, U2 to U1
Connections:
- net +3V3: now also C10.1, C11.1, C12.1, C13.1, C2.1, C3.1, C4.1, C5.1, C6.1, C7.1, C8.1, R2.2, U2.16 (VDD), U4.2 (VCC)
- net GND: now also C10.2, C11.2, C12.2, C13.2, C2.2, C3.2, C4.2, C5.2, C6.2, C7.2, C8.2, C?.1, D42.1 (K), D69.1 (K), R13.2, R14.2, R3.1, R4.1, R5.1, U2.8 (VSS), U4.29 (GND), U4.5 (GND)
- net GNSS_SCL: now also U2.1 (SCL), U4.20 (SCL)
- net GNSS_SDA: now also U2.2 (SDA), U4.19 (SDA)
- net GPIO[5]: now also R2.1, U2.15 (~{RESET})
- net ~{GNSS_RESET}: now also U2.6 (IO0)
- net ~{GNSS_SAFEBOOT}: now also U2.7 (IO1)
- net at R8.2: now also D42.2 (A)
- net at R9.2: now also D69.2 (A)
- net at C1.1, J1.1: now also C?.2, JP1.1 (A)
- net at L1.1: now also JP1.2 (B)
- new net: D11.2 (A), D19.2 (A), D3.2 (A), D37.2 (A), D46.2 (A), D54.2 (A), D62.2 (A)
- new net: D13.2 (A), D21.2 (A), D30.2 (A), D38.2 (A), D5.2 (A), D56.2 (A), D64.2 (A)
- new net: R3.2, U2.3 (A0)
- new net: D15.2 (A), D23.2 (A), D32.2 (A), D40.2 (A), D49.2 (A), D57.2 (A), D7.2 (A)
- new net: D14.2 (A), D22.2 (A), D31.2 (A), D39.2 (A), D48.2 (A), D6.2 (A), D65.2 (A)
- new net: D10.2 (A), D2.2 (A), D28.2 (A), D36.2 (A), D45.2 (A), D53.2 (A), D61.2 (A)
- new net: R14.1, U4.6 (R_EXT)
- new net: D12.2 (A), D20.2 (A), D29.2 (A), D4.2 (A), D47.2 (A), D55.2 (A), D63.2 (A)
- new net: R4.2, U2.4 (A1)
- new net: R5.2, U2.5 (A2)
- new net: R13.1, U4.18 (AD)
- new net CA1: D1.1 (K), D17.2 (A), D2.1 (K), D26.2 (A), D3.1 (K), D34.2 (A), D4.1 (K), D43.2 (A), D5.1 (K), D51.2 (A), D59.2 (A), D6.1 (K), D67.2 (A), D7.1 (K), D8.1 (K), D9.2 (A), U4.21 (CA1)
- new net CA2: D1.2 (A), D10.1 (K), D11.1 (K), D12.1 (K), D13.1 (K), D14.1 (K), D15.1 (K), D16.1 (K), D18.2 (A), D27.2 (A), D35.2 (A), D44.2 (A), D52.2 (A), D60.2 (A), D68.2 (A), D9.1 (K), U4.22 (CA2)
- new net CA3: D17.1 (K), D18.1 (K), D19.1 (K), D20.1 (K), D21.1 (K), D22.1 (K), D23.1 (K), D24.1 (K), U4.23 (CA3)
- new net CA4: D26.1 (K), D27.1 (K), D28.1 (K), D29.1 (K), D30.1 (K), D31.1 (K), D32.1 (K), D33.1 (K), U4.24 (CA4)
- new net CA5: D34.1 (K), D35.1 (K), D36.1 (K), D37.1 (K), D38.1 (K), D39.1 (K), D40.1 (K), D41.1 (K), U4.25 (CA5)
- new net CA6: D43.1 (K), D44.1 (K), D45.1 (K), D46.1 (K), D47.1 (K), D48.1 (K), D49.1 (K), D50.1 (K), U4.26 (CA6)
- new net CA7: D51.1 (K), D52.1 (K), D53.1 (K), D54.1 (K), D55.1 (K), D56.1 (K), D57.1 (K), D58.1 (K), U4.27 (CA7)
- new net CA8: D16.2 (A), D24.2 (A), D33.2 (A), D41.2 (A), D50.2 (A), D58.2 (A), D59.1 (K), D60.1 (K), D61.1 (K), D62.1 (K), D63.1 (K), D64.1 (K), D65.1 (K), D66.1 (K), D66.2 (A), D67.1 (K), D68.1 (K), D8.2 (A), U4.1 (CA9), U4.28 (CA8)
- new net ~{LEDMATRIX_INT}: U4.4 (~{INTB})
- new net ~{LEDMATRIX_OFF}: U2.9 (IO2), U4.3 (~{SDB})
- no-connect marks 6 -> 22
Other:
- note added: "66 channels (8x8+2)"
- note added: "GNSS channel indicator"
- note added: "GNSS receiver"
- note added: "GPIO connector"
- note added: "I2C expander"
- note added: "R added in case powered standalone"
- note added: "Raspberry Pi HAT EEPROM"
- note added: "address 0011xxx 0011000 / 0x18 / 24"
- note added: "default PU"
- moved on the sheet: BT1, C1, C14, C9, D25, J1, J2, J3, JP2, JP3, L1, R1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

Commit message: Update picise.kicad_sch
Connections:
- net ~{LEDMATRIX_INT}: now also U2.10 (IO3)
- no-connect marks 22 -> 21
Changed lines of the file:
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@@
   (no_connect (at 142.24 134.62))
   (no_connect (at 142.24 129.54))
-  (no_connect (at 142.24 127))
   (no_connect (at 124.46 220.98))
   (no_connect (at 124.46 238.76))
@@
     (stroke (width 0) (type default) (color 0 0 0 0))
   )
+  (wire (pts (xy 142.24 127) (xy 163.83 127))
+    (stroke (width 0) (type default) (color 0 0 0 0))
+  )
   (wire (pts (xy 166.37 187.96) (xy 166.37 200.66))
     (stroke (width 0) (type default) (color 0 0 0 0))
@@
     (effects (font (size 1.27 1.27)) (justify right bottom))
   )
+  (label "~{LEDMATRIX_INT}" (at 163.83 127 180)
+    (effects (font (size 1.27 1.27)) (justify right bottom))
+  )

Commit message: rev2 board prep
Parts:
- J2: footprint Connector_Header_Samtec:SAMTEC_SSQ-120-03-G-D_Pi_Annotated_PPS -> Connector_Header_Samtec:SAMTEC_SSQ-120-03-G-D_Pi
- J3: footprint Connector_PinHeader_2.54mm:PinHeader_1x02_P2.54mm_Vertical_SMD_Pin1Left -> Connector_PinHeader_2.54mm:PinHeader_1x02_P2.54mm_Vertical_SMD_Pin1Right
- JP1: value ACT_PSV -> TSM-103-01-L-SV; footprint (none) -> Connector_PinHeader_2.54mm:PinHeader_1x02_P2.54mm_Vertical_SMD_Pin1Right; Digikey (none) -> TSM-103-01-L-SV; MPN (none) -> TSM-102-01-L-SV; Manufacturer (none) -> Samtec
- gave numbers to parts that had none: 1
Changed lines of the file:
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@@
     (in_bom yes) (on_board yes)
     (property "Reference" "JP1" (id 0) (at 44.45 43.18 0))
-    (property "Value" "ACT_PSV" (id 1) (at 44.45 48.895 0))
-    (property "Footprint" "" (id 2) (at 44.45 45.72 0)
+    (property "Value" "TSM-103-01-L-SV" (id 1) (at 44.45 48.895 0))
+    (property "Footprint" "Connector_PinHeader_2.54mm:PinHeader_1x02_P2.54mm_Vertical_SMD_Pin1Right" (id 2) (at 44.45 45.72 0)
       (effects (font (size 1.27 1.27)) hide)
     )
     (property "Datasheet" "~" (id 3) (at 44.45 45.72 0)
+      (effects (font (size 1.27 1.27)) hide)
+    )
+    (property "Digikey" "TSM-103-01-L-SV" (id 4) (at 44.45 45.72 0)
+      (effects (font (size 1.27 1.27)) hide)
+    )
+    (property "MPN" "TSM-102-01-L-SV" (id 5) (at 44.45 45.72 0)
+      (effects (font (size 1.27 1.27)) hide)
+    )
+    (property "Manufacturer" "Samtec" (id 6) (at 44.45 45.72 0)
       (effects (font (size 1.27 1.27)) hide)
     )
@@
       (effects (font (size 1.27 1.27)) (justify left))
     )
-    (property "Footprint" "Connector_PinHeader_2.54mm:PinHeader_1x02_P2.54mm_Vertical_SMD_Pin1Left" (id 2) (at 284.48 265.43 0)
+    (property "Footprint" "Connector_PinHeader_2.54mm:PinHeader_1x02_P2.54mm_Vertical_SMD_Pin1Right" (id 2) (at 284.48 265.43 0)
       (effects (font (size 1.27 1.27)) hide)
     )
@@
   (symbol (lib_id "power:GND") (at 36.83 62.23 0) (unit 1)
     (in_bom yes) (on_board yes) (fields_autoplaced)
-    (property "Reference" "#PWR?" (id 0) (at 36.83 68.58 0)
+    (property "Reference" "#PWR0101" (id 0) (at 36.83 68.58 0)
       (effects (font (size 1.27 1.27)) hide)
     )
@@
   (symbol (lib_id "Connector_Header_Samtec:SSQ-120-03_GPIO") (at 335.28 62.23 0) (unit 1)
     (in_bom yes) (on_board yes) (fields_autoplaced)
-    (property "Reference" "J2" (id 0) (at 327.152 34.29 0)
-      (effects (font (size 1.27 1.27)) (justify left bottom))
-    )
-    (property "Value" "SSQ-120-03_GPIO" (id 1) (at 326.39 90.17 0)
-      (effects (font (size 1.27 1.27)) (justify left bottom))
-    )
-    (property "Footprint" "Connector_Header_Samtec:SAMTEC_SSQ-120-03-G-D_Pi_Annotated_PPS" (id 2) (at 320.04 100.965 0)
+    (property "Reference" "J2" (id 0) (at 335.28 29.21 0))
+    (property "Value" "SSQ-120-03_GPIO" (id 1) (at 335.28 31.75 0))
+    (property "Footprint" "Connector_Header_Samtec:SAMTEC_SSQ-120-03-G-D_Pi" (id 2) (at 320.04 100.965 0)
       (effects (font (size 1.27 1.27)) (justify left bottom) hide)
     )
@@
   (symbol (lib_id "Device:C_Small") (at 36.83 54.61 180) (unit 1)
     (in_bom yes) (on_board yes)
-    (property "Reference" "C?" (id 0) (at 40.64 53.34 0))
+    (property "Reference" "C15" (id 0) (at 40.64 53.34 0))
     (property "Value" "22pF" (id 1) (at 41.91 55.88 0))
     (property "Footprint" "Capacitor_SMD:C_0603_1608Metric" (id 2) (at 36.83 54.61 0)
@@
     )
     (path "/cdb19993-fb1f-4de5-8403-e02eb54bbf92"
-      (reference "#PWR?") (unit 1) (value "GND") (footprint "")
+      (reference "#PWR0101") (unit 1) (value "GND") (footprint "")
     )
     (path "/bafff22c-8857-4139-9e66-e6877e94d1c3"
@@
     )
     (path "/f95f0a99-19ab-4e4f-a6a3-759367232c47"
-      (reference "C?") (unit 1) (value "22pF") (footprint "Capacitor_SMD:C_0603_1608Metric")
+      (reference "C15") (unit 1) (value "22pF") (footprint "Capacitor_SMD:C_0603_1608Metric")
     )
     (path "/72ea6034-c134-406a-b932-15997193ab7c"
@@
     )
     (path "/df883408-807c-458f-924a-53ad59baf3c9"
-      (reference "J2") (unit 1) (value "SSQ-120-03_GPIO") (footprint "Connector_Header_Samtec:SAMTEC_SSQ-120-03-G-D_Pi_Annotated_PPS")
+      (reference "J2") (unit 1) (value "SSQ-120-03_GPIO") (footprint "Connector_Header_Samtec:SAMTEC_SSQ-120-03-G-D_Pi")
     )
     (path "/b5bc33c5-f237-4113-82dc-9833ded1e077"
-      (reference "J3") (unit 1) (value "TSM-103-01-L-SV") (footprint "Connector_PinHeader_2.54mm:PinHeader_1x02_P2.54mm_Vertical_SMD_Pin1Left")
+      (reference "J3") (unit 1) (value "TSM-103-01-L-SV") (footprint "Connector_PinHeader_2.54mm:PinHeader_1x02_P2.54mm_Vertical_SMD_Pin1Right")
     )
     (path "/adfb47a7-7a6e-463b-99e4-7ee8fae51556"
-      (reference "JP1") (unit 1) (value "ACT_PSV") (footprint "")
+      (reference "JP1") (unit 1) (value "TSM-103-01-L-SV") (footprint "Connector_PinHeader_2.54mm:PinHeader_1x02_P2.54mm_Vertical_SMD_Pin1Right")
     )
     (path "/43e66c4c-de75-44f8-8171-19825b035cbb"

Commit message: rev2 prep
Parts:
- added D70, D71, D72, D73, D74, D75: Green, Diode_SMD:D_0603_1608Metric, symbol Device:LED_Small_Filled
Connections:
- net CA3: now also D10.2 (A), D2.2 (A), D28.2 (A), D36.2 (A), D45.2 (A), D53.2 (A), D61.2 (A), D70.2 (A)
- net CA4: now also D11.2 (A), D19.2 (A), D3.2 (A), D37.2 (A), D46.2 (A), D54.2 (A), D62.2 (A), D71.2 (A)
- net CA5: now also D12.2 (A), D20.2 (A), D29.2 (A), D4.2 (A), D47.2 (A), D55.2 (A), D63.2 (A), D72.2 (A)
- net CA6: now also D13.2 (A), D21.2 (A), D30.2 (A), D38.2 (A), D5.2 (A), D56.2 (A), D64.2 (A), D73.2 (A)
- net CA7: now also D14.2 (A), D22.2 (A), D31.2 (A), D39.2 (A), D48.2 (A), D6.2 (A), D65.2 (A), D74.2 (A)
- net CA8: now also D15.2 (A), D23.2 (A), D32.2 (A), D40.2 (A), D49.2 (A), D57.2 (A), D7.2 (A), D70.1 (K), D71.1 (K), D72.1 (K), D73.1 (K), D74.1 (K), D75.1 (K), D75.2 (A)
Other:
- note added: "66 channels (8x9)"
- note removed: "66 channels (8x8+2)"

Commit message: rev2 prep
Parts:
- removed C10, C11: 10uF, Capacitor_SMD:C_0603_1608Metric, symbol Device:C_Small
- removed C12: 1uF, Capacitor_SMD:C_0603_1608Metric, symbol Device:C_Small
- removed C13: 0.1uF, Capacitor_SMD:C_0603_1608Metric, symbol Device:C_Small
- removed D1, D10, D11, D12, D13, D14, D15, D16, D17, D18, D19, D2, D20, D21, D22, D23, D24, D26, D27, D28, D29, D3, D30, D31, D32, D33, D34, D35, D36, D37, D38, D39, D4, D40, D41, D43, D44, D45, D46, D47, D48, D49, D5, D50, D51, D52, D53, D54, D55, D56, D57, D58, D59, D6, D60, D61, D62, D63, D64, D65, D66, D67, D68, D7, D70, D71, D72, D73, D74, D75, D8, D9: Green, Diode_SMD:D_0603_1608Metric, symbol Device:LED_Small_Filled
- removed R13, R14: 20k, Resistor_SMD:R_0603_1608Metric, symbol Device:R_Small
- removed U4: IS31FL3731-QF, Package_DFN_QFN:QFN-28-1EP_4x4mm_P0.4mm_EP2.3x2.3mm, symbol Driver_LED:IS31FL3731-QF
Connections:
- no-connect marks 21 -> 10
Other:
- note added: "Status Display"
- note removed: "66 channels (8x9)"
- note removed: "GNSS channel indicator"
