File: picise.kicad_sch (KiCad schematic)
At the start: 37 parts, among them J1 ANT_SMA, J2 SSQ-120-03_GPIO, J3 TSM-103-01-L-SV, U1 MAX-M10S, U2 PCA9557PW, U3 CAT24C256

Commit message: rev2 prep
Parts:
- added DS1: NHD-C12832A1Z-FSW-FBW-3V3, Display_LCD_Newhaven:LCD_NHD-C12832A1Z-FSW-FBW-3V3, symbol Display_LCD_Newhaven:NHD-C12832A1Z-FSW-FBW-3V3
Connections:
- net GPIO[10]/SPI0.MOSI renamed DISP_MOSI
- net DISP_MOSI: now also DS1.13 (SI)
- net GPIO[11]/SPI0.SCLK renamed DISP_SCLK
- net DISP_SCLK: now also DS1.14 (SCL)
- net GPIO[8]/SPI0.CE0 renamed DISP_CE0
- net DISP_CE0: now also DS1.17 (~{CS1})
- net ~{LEDMATRIX_INT}: no longer names the net of U2.10 (IO3)
- net ~{LEDMATRIX_OFF} renamed ~{DISP_RST}
- net ~{DISP_RST}: now also DS1.16 (~{RST})
Changed lines of the file:
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@@
     (stroke (width 0) (type default) (color 0 0 0 0))
   )
-  (wire (pts (xy 293.37 64.77) (xy 322.58 64.77))
+  (wire (pts (xy 273.05 64.77) (xy 322.58 64.77))
     (stroke (width 0) (type solid) (color 0 0 0 0))
   )
@@
     (stroke (width 0) (type default) (color 0 0 0 0))
   )
+  (wire (pts (xy 95.25 212.09) (xy 106.68 212.09))
+    (stroke (width 0) (type default) (color 0 0 0 0))
+  )
   (wire (pts (xy 322.58 49.53) (xy 293.37 49.53))
     (stroke (width 0) (type solid) (color 0 0 0 0))
@@
     (stroke (width 0) (type default) (color 0 0 0 0))
   )
+  (wire (pts (xy 95.25 252.73) (xy 106.68 252.73))
+    (stroke (width 0) (type default) (color 0 0 0 0))
+  )
   (wire (pts (xy 350.52 41.91) (xy 347.98 41.91))
     (stroke (width 0) (type solid) (color 0 0 0 0))
@@
     (stroke (width 0) (type solid) (color 0 0 0 0))
   )
+  (wire (pts (xy 95.25 207.01) (xy 106.68 207.01))
+    (stroke (width 0) (type default) (color 0 0 0 0))
+  )
   (wire (pts (xy 101.6 120.65) (xy 101.6 124.46))
     (stroke (width 0) (type default) (color 0 0 0 0))
@@
     (stroke (width 0) (type solid) (color 0 0 0 0))
   )
+  (wire (pts (xy 347.98 64.77) (xy 394.97 64.77))
+    (stroke (width 0) (type default) (color 0 0 0 0))
+  )
   (wire (pts (xy 322.58 200.66) (xy 334.01 200.66))
     (stroke (width 0) (type default) (color 0 0 0 0))
   )
+  (wire (pts (xy 48.26 227.33) (xy 59.69 227.33))
+    (stroke (width 0) (type default) (color 0 0 0 0))
+  )
   (wire (pts (xy 68.58 111.76) (xy 68.58 115.57))
     (stroke (width 0) (type default) (color 0 0 0 0))
@@
     (stroke (width 0) (type default) (color 0 0 0 0))
   )
-  (wire (pts (xy 347.98 64.77) (xy 374.65 64.77))
-    (stroke (width 0) (type solid) (color 0 0 0 0))
-  )
   (wire (pts (xy 106.68 38.1) (xy 106.68 40.64))
     (stroke (width 0) (type default) (color 0 0 0 0))
@@
     (stroke (width 0) (type default) (color 0 0 0 0))
   )
+  (wire (pts (xy 95.25 214.63) (xy 106.68 214.63))
+    (stroke (width 0) (type default) (color 0 0 0 0))
+  )
   (wire (pts (xy 132.08 114.3) (xy 132.08 111.76))
     (stroke (width 0) (type default) (color 0 0 0 0))
@@
     (stroke (width 0) (type solid) (color 0 0 0 0))
   )
-  (wire (pts (xy 322.58 59.69) (xy 293.37 59.69))
+  (wire (pts (xy 273.05 59.69) (xy 322.58 59.69))
     (stroke (width 0) (type solid) (color 0 0 0 0))
   )
@@
     (stroke (width 0) (type solid) (color 0 0 0 0))
   )
+  (wire (pts (xy 95.25 232.41) (xy 106.68 232.41))
+    (stroke (width 0) (type default) (color 0 0 0 0))
+  )
   (wire (pts (xy 273.05 72.39) (xy 322.58 72.39))
     (stroke (width 0) (type default) (color 0 0 0 0))
@@
     (stroke (width 0) (type default) (color 0 0 0 0))
   )
+  (wire (pts (xy 48.26 240.03) (xy 59.69 240.03))
+    (stroke (width 0) (type default) (color 0 0 0 0))
+  )
   (wire (pts (xy 368.3 144.78) (xy 368.3 147.32))
     (stroke (width 0) (type solid) (color 0 0 0 0))
@@
     (stroke (width 0) (type solid) (color 0 0 0 0))
   )
+  (wire (pts (xy 95.25 219.71) (xy 106.68 219.71))
+    (stroke (width 0) (type default) (color 0 0 0 0))
+  )
   (wire (pts (xy 320.04 229.87) (xy 320.04 234.95))
     (stroke (width 0) (type default) (color 0 0 0 0))
@@
     (stroke (width 0) (type default) (color 0 0 0 0))
   )
+  (wire (pts (xy 95.25 227.33) (xy 106.68 227.33))
+    (stroke (width 0) (type default) (color 0 0 0 0))
+  )
   (wire (pts (xy 71.12 50.8) (xy 71.12 55.88))
     (stroke (width 0) (type default) (color 0 0 0 0))
@@
     (stroke (width 0) (type default) (color 0 0 0 0))
   )
+  (wire (pts (xy 95.25 217.17) (xy 106.68 217.17))
+    (stroke (width 0) (type default) (color 0 0 0 0))
+  )
+  (wire (pts (xy 95.25 234.95) (xy 106.68 234.95))
+    (stroke (width 0) (type default) (color 0 0 0 0))
+  )
   (wire (pts (xy 320.04 234.95) (xy 328.93 234.95))
     (stroke (width 0) (type default) (color 0 0 0 0))
@@
     (stroke (width 0) (type default) (color 0 0 0 0))
   )
+  (wire (pts (xy 95.25 240.03) (xy 106.68 240.03))
+    (stroke (width 0) (type default) (color 0 0 0 0))
+  )
   (wire (pts (xy 337.82 137.16) (xy 337.82 147.32))
     (stroke (width 0) (type solid) (color 0 0 0 0))
@@
     (stroke (width 0) (type default) (color 0 0 0 0))
   )
+  (wire (pts (xy 95.25 247.65) (xy 106.68 247.65))
+    (stroke (width 0) (type default) (color 0 0 0 0))
+  )
   (polyline (pts (xy 299.72 187.96) (xy 262.89 187.96))
     (stroke (width 0) (type default) (color 0 0 0 0))
@@
     (stroke (width 0) (type default) (color 0 0 0 0))
   )
+  (wire (pts (xy 95.25 222.25) (xy 106.68 222.25))
+    (stroke (width 0) (type default) (color 0 0 0 0))
+  )
+  (wire (pts (xy 48.26 237.49) (xy 59.69 237.49))
+    (stroke (width 0) (type default) (color 0 0 0 0))
+  )
+  (wire (pts (xy 95.25 245.11) (xy 106.68 245.11))
+    (stroke (width 0) (type default) (color 0 0 0 0))
+  )
   (wire (pts (xy 289.56 218.44) (xy 290.83 218.44))
     (stroke (width 0) (type default) (color 0 0 0 0))
@@
   )
   (wire (pts (xy 328.93 245.11) (xy 328.93 234.95))
+    (stroke (width 0) (type default) (color 0 0 0 0))
+  )
+  (wire (pts (xy 48.26 242.57) (xy 59.69 242.57))
+    (stroke (width 0) (type default) (color 0 0 0 0))
+  )
+  (wire (pts (xy 48.26 232.41) (xy 59.69 232.41))
+    (stroke (width 0) (type default) (color 0 0 0 0))
+  )
+  (wire (pts (xy 95.25 237.49) (xy 106.68 237.49))
     (stroke (width 0) (type default) (color 0 0 0 0))
   )
@@
     (effects (font (size 1.27 1.27)) (justify left bottom))
   )
+  (label "~{DISP_RST}" (at 163.83 124.46 180)
+    (effects (font (size 1.27 1.27)) (justify right bottom))
+  )
   (label "GPIO[23]" (at 374.65 54.61 180)
     (effects (font (size 1.27 1.27)) (justify right bottom))
@@
     (effects (font (size 1.27 1.27)) (justify right bottom))
   )
+  (label "DISP_SCLK" (at 48.26 237.49 0)
+    (effects (font (size 1.27 1.27)) (justify left bottom))
+  )
   (label "GNSS_SDA" (at 52.07 55.88 0)
     (effects (font (size 1.27 1.27)) (justify left bottom))
   )
+  (label "DISP_MOSI" (at 48.26 240.03 0)
+    (effects (font (size 1.27 1.27)) (justify left bottom))
+  )
   (label "GPIO[17]" (at 293.37 49.53 0)
     (effects (font (size 1.27 1.27)) (justify left bottom))
@@
     (effects (font (size 1.27 1.27)) (justify left bottom))
   )
+  (label "DISP_CE0" (at 394.97 64.77 180)
+    (effects (font (size 1.27 1.27)) (justify right bottom))
+  )
   (label "GPIO[13]{slash}PWM1" (at 293.37 77.47 0)
     (effects (font (size 1.27 1.27)) (justify left bottom))
   )
+  (label "~{DISP_RST}" (at 48.26 227.33 0)
+    (effects (font (size 1.27 1.27)) (justify left bottom))
+  )
   (label "GPIO[8]{slash}SPI0.CE0" (at 374.65 64.77 180)
     (effects (font (size 1.27 1.27)) (justify right bottom))
@@
     (effects (font (size 1.27 1.27)) (justify left bottom))
   )
+  (label "DISP_SCLK" (at 273.05 64.77 0)
+    (effects (font (size 1.27 1.27)) (justify left bottom))
+  )
   (label "~{GNSS_SAFEBOOT}" (at 52.07 60.96 0)
     (effects (font (size 1.27 1.27)) (justify left bottom))
@@
     (effects (font (size 1.27 1.27)) (justify left bottom))
   )
+  (label "DISP_MOSI" (at 273.05 59.69 0)
+    (effects (font (size 1.27 1.27)) (justify left bottom))
+  )
   (label "ID_SCL" (at 374.65 69.85 180)
     (effects (font (size 1.27 1.27)) (justify right bottom))
@@
     (effects (font (size 1.27 1.27)) (justify right bottom))
   )
-  (label "~{LEDMATRIX_INT}" (at 163.83 127 180)
-    (effects (font (size 1.27 1.27)) (justify right bottom))
-  )
-  (label "~{LEDMATRIX_OFF}" (at 163.83 124.46 180)
-    (effects (font (size 1.27 1.27)) (justify right bottom))
-  )
   (label "GPIO[18]{slash}PCM.CLK" (at 374.65 49.53 180)
     (effects (font (size 1.27 1.27)) (justify right bottom))
+  )
+  (label "DISP_CE0" (at 48.26 242.57 0)
+    (effects (font (size 1.27 1.27)) (justify left bottom))
   )
   (label "GNSS_TX" (at 394.97 46.99 180)
@@
     (pin "2")
     (pin "3")
+  )
+  (symbol (lib_id "Display_LCD_Newhaven:NHD-C12832A1Z-FSW-FBW-3V3") (at 77.47 229.87 0) (unit 1)
+    (in_bom yes) (on_board yes) (fields_autoplaced)
+    (property "Reference" "DS1" (id 0) (at 77.47 199.39 0))
+    (property "Value" "NHD-C12832A1Z-FSW-FBW-3V3" (id 1) (at 77.47 201.93 0))
+    (property "Footprint" "Display_LCD_Newhaven:LCD_NHD-C12832A1Z-FSW-FBW-3V3" (id 2) (at 50.8 269.24 0)
+      (effects (font (size 1.27 1.27)) (justify left bottom) hide)
+    )
+    (property "Datasheet" "" (id 3) (at 77.47 229.87 0)
+      (effects (font (size 1.27 1.27)) (justify left bottom) hide)
+    )
+    (property "Manufacturer" "Newhaven" (id 6) (at 73.025 265.43 0)
+      (effects (font (size 1.27 1.27)) (justify left bottom) hide)
+    )
+    (property "MPN" "NHD-C12832A1Z-FSW-FBW-3V3" (id 8) (at 78.105 274.32 0)
+      (effects (font (size 1.27 1.27)) hide)
+    )
+    (pin "1")
+    (pin "10")
+    (pin "11")
+    (pin "12")
+    (pin "13")
+    (pin "14")
+    (pin "15")
+    (pin "16")
+    (pin "17")
+    (pin "2")
+    (pin "3")
+    (pin "4")
+    (pin "5")
+    (pin "6")
+    (pin "7")
+    (pin "8")
+    (pin "9")
+    (pin "A")
+    (pin "K")
   )
   (symbol (lib_id "power:GND") (at 106.68 62.23 0) (unit 1)
@@
       (reference "D69") (unit 1) (value "Blue") (footprint "Diode_SMD:D_0603_1608Metric")
     )
+    (path "/4ae6dfb3-4f43-4c55-a4ca-fc9d674901ab"
+      (reference "DS1") (unit 1) (value "NHD-C12832A1Z-FSW-FBW-3V3") (footprint "Display_LCD_Newhaven:LCD_NHD-C12832A1Z-FSW-FBW-3V3")
+    )
     (path "/e38330bb-c7ad-4477-8444-fab35c01fdca"

Commit message: rev2 prep
Parts:
- removed DS1: NHD-C12832A1Z-FSW-FBW-3V3, Display_LCD_Newhaven:LCD_NHD-C12832A1Z-FSW-FBW-3V3, symbol Display_LCD_Newhaven:NHD-C12832A1Z-FSW-FBW-3V3
- added DS1: NHD-3.12-25664UCB2_SPI, Display_OLED_Newhaven:OLED_NHD-3.12-25664UCx2, symbol Display_OLED_Newhaven:NHD-3.12-25664UCB2_SPI
Connections:
- net +3V3: now also DS1.2 (VDD)
- net DISP_MOSI: now also DS1.7 (SDIN)
- net DISP_SCLK: now also DS1.6 (SCLK)
- net GND: now also DS1.1 (VSS), DS1.10 (VSS), DS1.11 (VSS), DS1.12 (VSS), DS1.13 (VSS), DS1.14 (VSS), DS1.19 (BS1), DS1.20 (BS2), DS1.5 (VSS), DS1.9 (VSS)
- net ~{DISP_RST}: now also DS1.16 (~{RST})
- net DISP_CE0 renamed GPIO[8]/SPI0.CE0
- net GPIO[8]/SPI0.CE0: now also DS1.17 (~{CS})
- net GPIO[26] renamed DISP_D_C
- net DISP_D_C: now also DS1.4 (D/C)
- new net: DS1.15 (NC), DS1.18 (NC), DS1.3 (NC), DS1.8 (NC)

Commit message: rev2 draft routed
Parts:
- removed J3: TSM-103-01-L-SV, Connector_PinHeader_2.54mm:PinHeader_1x02_P2.54mm_Vertical_SMD_Pin1Right, symbol Connector_Generic:Conn_01x02
- removed JP1: TSM-103-01-L-SV, Connector_PinHeader_2.54mm:PinHeader_1x02_P2.54mm_Vertical_SMD_Pin1Right, symbol Jumper:Jumper_2_Bridged
- added C10, C11: 10uF, Capacitor_SMD:C_0603_1608Metric, symbol Device:C_Small
- added C12: 1uF, Capacitor_SMD:C_0603_1608Metric, symbol Device:C_Small
- added C13: 0.1uF, Capacitor_SMD:C_0603_1608Metric, symbol Device:C_Small
Connections:
- net +3V3: now also C10.1, C11.1, C12.1, C13.1
- net GND: now also C10.2, C11.2, C12.2, C13.2
- net at C1.1, C15.2, J1.1: now also L1.1
Other:
- note removed: "Fan header"
- moved on the sheet: BT1, C14, D25, D42, D69, DS1, JP3, R10, R11, R12, R8, R9

Commit message: tweaks
Parts:
- removed C10, C11: 10uF, Capacitor_SMD:C_0603_1608Metric, symbol Device:C_Small
- removed C12: 1uF, Capacitor_SMD:C_0603_1608Metric, symbol Device:C_Small
- removed C13: 0.1uF, Capacitor_SMD:C_0603_1608Metric, symbol Device:C_Small
- removed DS1: NHD-3.12-25664UCB2_SPI, Display_OLED_Newhaven:OLED_NHD-3.12-25664UCx2, symbol Display_OLED_Newhaven:NHD-3.12-25664UCB2_SPI
Connections:
- net DISP_D_C renamed GPIO[26]
- net DISP_MOSI renamed GPIO[10]/SPI0.MOSI
- net DISP_SCLK renamed GPIO[11]/SPI0.SCLK
- net ~{DISP_RST}: no longer names the net of U2.9 (IO2)
- no-connect marks 10 -> 12
Other:
- note removed: "Status Display"
- moved on the sheet: BT1, C1, C14, C15, C2, C3, C4, C5, C6, C7, C8, C9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
