File: picise.kicad_pcb (KiCad board)
At the start: 2 copper layers, 65 x 76 mm, 26 parts, among them J1 SSW-120-22-G-D-RA, J2 SMA jack, J3 TSW-120-08-G-D-RA, J4 Conn_01x02, U1 CAT24C256, U2 MAX-M10S

Commit message: rev2 prep
Parts:
- moved C3 1.36 mm to (155.6, 76.8), turned to 180 degrees
Routing:
- net GND: track 608.3 -> 609.9 mm
- net +3V3: track 210.7 -> 209.3 mm
Changed lines of the file:
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@@
   (title_block
     (date "15 nov 2012")
+    (rev "2")
   )
   (layers
@@
   )
   (footprint "Capacitor_SMD:C_0805_2012Metric_Pad1.18x1.45mm_HandSolder" (layer "B.Cu")
-    (at 156.9 77.2 135)
+    (at 155.6 76.8 180)
     (descr "Capacitor SMD 0805 (2012 Metric), square (rectangular) end terminal, IPC_7351 nominal with elongated pad for handsoldering. (Body size source: IPC-SM-782 page 76, https://www.pcb-3d.com/wordpress/wp-content/uploads/ipc-sm-782a_amendment_1_and_2.pdf, https://docs.google.com/spreadsheets/d/1BsfQQcO9C6DZCsRaXUlFlo91Tg2WpOkGARC1WS5S8t0/edit?usp=sharing), generated with kicad-footprint-generator")
     (tags "capacitor handsolder")
@@
     (property "Sheetname" "")
     (attr smd)
-    (fp_text reference "C3" (at 0 1.68 135) (layer "B.SilkS") hide
-      (effects (font (size 1 1) (thickness 0.15)) (justify mirror))
-    )
-    (fp_text value "22pF" (at 0 -1.68 135) (layer "B.Fab")
-      (effects (font (size 1 1) (thickness 0.15)) (justify mirror))
-    )
-    (fp_text user "${REFERENCE}" (at 0 0 135) (layer "B.Fab")
+    (fp_text reference "C3" (at 0 1.68) (layer "B.SilkS") hide
+      (effects (font (size 1 1) (thickness 0.15)) (justify mirror))
+    )
+    (fp_text value "22pF" (at 0 -1.68) (layer "B.Fab")
+      (effects (font (size 1 1) (thickness 0.15)) (justify mirror))
+    )
+    (fp_text user "${REFERENCE}" (at 0 0) (layer "B.Fab")
       (effects (font (size 0.5 0.5) (thickness 0.08)) (justify mirror))
     )
@@
     (fp_line (start 1 -0.625) (end -1 -0.625) (layer "B.Fab") (width 0.1))
     (fp_line (start -1 -0.625) (end -1 0.625) (layer "B.Fab") (width 0.1))
-    (pad "1" smd roundrect (at -1.0375 0 135) (size 1.175 1.45) (layers "B.Cu" "B.Paste" "B.Mask") (roundrect_rratio 0.2127659574)
+    (pad "1" smd roundrect (at -1.0375 0 180) (size 1.175 1.45) (layers "B.Cu" "B.Paste" "B.Mask") (roundrect_rratio 0.2127659574)
       (net 1 "GND") (pintype "passive"))
-    (pad "2" smd roundrect (at 1.0375 0 135) (size 1.175 1.45) (layers "B.Cu" "B.Paste" "B.Mask") (roundrect_rratio 0.2127659574)
+    (pad "2" smd roundrect (at 1.0375 0 180) (size 1.175 1.45) (layers "B.Cu" "B.Paste" "B.Mask") (roundrect_rratio 0.2127659574)
       (net 28 "+3V3") (pintype "passive"))
     (model "${KICAD6_3DMODEL_DIR}/Capacitor_SMD.3dshapes/C_0805_2012Metric.wrl"
@@
   (via (at 117 107.4) (size 0.9) (drill 0.6) (layers "F.Cu" "B.Cu") (free) (net 1))
   (segment (start 126.75 84.35) (end 129.75 84.35) (width 0.4) (layer "B.Cu") (net 1))
+  (segment (start 156.6375 76.8) (end 156.6375 78.6875) (width 0.7) (layer "B.Cu") (net 1))
   (segment (start 159.6505 79.8) (end 159.75 79.7005) (width 0.7) (layer "B.Cu") (net 1))
-  (segment (start 157.633623 77.933623) (end 157.633623 79.683623) (width 0.7) (layer "B.Cu") (net 1))
   (segment (start 161.225 78.075) (end 162.9 78.075) (width 0.7) (layer "B.Cu") (net 1))
-  (segment (start 157.633623 79.683623) (end 157.75 79.8) (width 0.7) (layer "B.Cu") (net 1))
   (segment (start 157.75 82) (end 159.6505 82) (width 0.7) (layer "B.Cu") (net 1))
   (segment (start 148.25 88.6) (end 146.4 88.6) (width 0.7) (layer "B.Cu") (net 1))
@@
   (segment (start 161.125 83.725) (end 162.9 83.725) (width 0.7) (layer "B.Cu") (net 1))
   (segment (start 159.75 79.55) (end 161.225 78.075) (width 0.7) (layer "B.Cu") (net 1))
+  (segment (start 156.6375 78.6875) (end 157.75 79.8) (width 0.7) (layer "B.Cu") (net 1))
   (segment (start 122.9625 82.1625) (end 122.9625 82.55) (width 0.7) (layer "B.Cu") (net 1))
   (segment (start 124.5625 82.1625) (end 126.75 84.35) (width 0.4) (layer "B.Cu") (net 1))
@@
   (via (at 125.21 79.8) (size 1) (drill 0.7) (layers "F.Cu" "B.Cu") (net 28))
   (segment (start 147.424695 80.9) (end 148.25 80.9) (width 0.7) (layer "B.Cu") (net 28))
+  (segment (start 154.4 76.9625) (end 154.5625 76.8) (width 0.7) (layer "B.Cu") (net 28))
   (segment (start 138.03 110.4525) (end 140.0475 112.47) (width 0.7) (layer "B.Cu") (net 28))
   (segment (start 135.29 108.36) (end 137.83 108.36) (width 0.7) (layer "B.Cu") (net 28))
@@
   (segment (start 125.2 96.71) (end 125.2 98.4575) (width 0.7) (layer "B.Cu") (net 28))
   (segment (start 138.03 110.4525) (end 137.845 110.2675) (width 0.7) (layer "B.Cu") (net 28))
-  (segment (start 154.4 77.6) (end 155.533623 76.466377) (width 0.7) (layer "B.Cu") (net 28))
   (segment (start 140.0475 112.47) (end 140.4 112.47) (width 0.7) (layer "B.Cu") (net 28))
   (segment (start 137.845 110.2675) (end 137.845 108.345) (width 0.7) (layer "B.Cu") (net 28))
@@
   (segment (start 127.6525 79.8) (end 127.6575 79.805) (width 0.7) (layer "B.Cu") (net 28))
   (segment (start 135.29 108.36) (end 125.26 108.36) (width 0.7) (layer "B.Cu") (net 28))
-  (segment (start 154.4 78.3) (end 154.4 77.6) (width 0.7) (layer "B.Cu") (net 28))
+  (segment (start 154.4 78.3) (end 154.4 76.9625) (width 0.7) (layer "B.Cu") (net 28))
   (segment (start 125.21 96.7) (end 125.2 96.71) (width 0.7) (layer "B.Cu") (net 28))
-  (segment (start 155.533623 76.466377) (end 156.166377 76.466377) (width 0.7) (layer "B.Cu") (net 28))
   (segment (start 127.6575 79.805) (end 146.329695 79.805) (width 0.7) (layer "B.Cu") (net 28))
   (segment (start 146.329695 79.805) (end 147.424695 80.9) (width 0.7) (layer "B.Cu") (net 28))
@@
   (segment (start 157.75 80.9) (end 156.712563 80.9) (width 1) (layer "B.Cu") (net 42))
   (segment (start 157.75 80.9) (end 163.1 80.9) (width 1) (layer "B.Cu") (net 42))
-  (segment (start 155.45 79.637437) (end 155.45 78.4) (width 1) (layer "B.Cu") (net 42))
   (segment (start 156.712563 80.9) (end 155.45 79.637437) (width 1) (layer "B.Cu") (net 42))
+  (segment (start 155.45 79.637437) (end 155.45 78.3) (width 1) (layer "B.Cu") (net 42))
   (segment (start 109.6675 114.2) (end 109.62 114.2) (width 0.2) (layer "F.Cu") (net 43))
   (segment (start 110.93 115.46) (end 109.67 114.2) (width 0.7) (layer "F.Cu") (net 43))

Commit message: rev2 board prep
Parts:
- removed J4: Conn_01x02, Connector_PinHeader_2.54mm:PinHeader_1x02_P2.54mm_Vertical_SMD_Pin1Left
- added C10: 10uF, Capacitor_SMD:C_0603_1608Metric, F.Cu at (-46.1, 74.3)
- added C11: 10uF, Capacitor_SMD:C_0603_1608Metric, F.Cu at (-33.5, 71.8)
- added C12: 1uF, Capacitor_SMD:C_0603_1608Metric, F.Cu at (-50.2, 74.3)
- added C13: 0.1uF, Capacitor_SMD:C_0603_1608Metric, F.Cu at (-38.2, 76.8)
- added C14: 1uF, Capacitor_SMD:C_0603_1608Metric, F.Cu at (-49.5, 71.8)
- added C15: 22pF, Capacitor_SMD:C_0603_1608Metric, F.Cu at (-50.1, 79.3)
- added C4: 0.1uF, Capacitor_SMD:C_0603_1608Metric, F.Cu at (-54.2, 74.3)
- added C5: 10uF, Capacitor_SMD:C_0603_1608Metric, F.Cu at (-50.2, 76.8)
- added C6: 10uF, Capacitor_SMD:C_0603_1608Metric, F.Cu at (-62.1, 79.3)
- added C7: 1uF, Capacitor_SMD:C_0603_1608Metric, F.Cu at (-41.5, 71.8)
- added C8: 0.1uF, Capacitor_SMD:C_0603_1608Metric, F.Cu at (-34.1, 74.3)
- added C9: 0.1uF, Capacitor_SMD:C_0603_1608Metric, F.Cu at (-53.5, 71.8)
- added D10: Green, Diode_SMD:D_0603_1608Metric, F.Cu at (82.0, 81.5)
- added D11: Green, Diode_SMD:D_0603_1608Metric, F.Cu at (24.4, 98.4)
- added D12: Green, Diode_SMD:D_0603_1608Metric, F.Cu at (41.3, 93.9)
- added D13: Green, Diode_SMD:D_0603_1608Metric, F.Cu at (16.5, 106.2)
- added D14: Green, Diode_SMD:D_0603_1608Metric, F.Cu at (98.2, 80.7)
- added D15: Green, Diode_SMD:D_0603_1608Metric, F.Cu at (86.0, 84.1)
- added D16: Green, Diode_SMD:D_0603_1608Metric, F.Cu at (41.0, 89.7)
- added D17: Green, Diode_SMD:D_0603_1608Metric, F.Cu at (45.4, 93.9)
- added D18: Green, Diode_SMD:D_0603_1608Metric, F.Cu at (78.0, 86.7)
- added D19: Green, Diode_SMD:D_0603_1608Metric, F.Cu at (73.9, 86.7)
- added D20: Green, Diode_SMD:D_0603_1608Metric, F.Cu at (69.8, 82.5)
- added D21: Green, Diode_SMD:D_0603_1608Metric, F.Cu at (94.2, 83.3)
- added D22: Green, Diode_SMD:D_0603_1608Metric, F.Cu at (68.7, 89.3)
- added D23: Green, Diode_SMD:D_0603_1608Metric, F.Cu at (20.8, 85.0)
- added D24: Green, Diode_SMD:D_0603_1608Metric, F.Cu at (16.5, 103.6)
- added D25: 0.5A 40V 420mV, Diode_SMD:D_0603_1608Metric, F.Cu at (90.1, 85.9)
- added D26: Green, Diode_SMD:D_0603_1608Metric, F.Cu at (72.8, 89.3)
- added D27: Green, Diode_SMD:D_0603_1608Metric, F.Cu at (37.2, 93.9)
- added D28: Green, Diode_SMD:D_0603_1608Metric, F.Cu at (12.4, 107.6)
- added D29: Green, Diode_SMD:D_0603_1608Metric, F.Cu at (94.2, 80.7)
- added D3: Green, Diode_SMD:D_0603_1608Metric, F.Cu at (8.40, 105.0)
- added D30: Green, Diode_SMD:D_0603_1608Metric, F.Cu at (28.9, 89.7)
- added D31: Green, Diode_SMD:D_0603_1608Metric, F.Cu at (8.40, 107.6)
- added D32: Green, Diode_SMD:D_0603_1608Metric, F.Cu at (87.6, 76.3)
- added D33: Green, Diode_SMD:D_0603_1608Metric, F.Cu at (84.9, 89.3)
- added D34: Green, Diode_SMD:D_0603_1608Metric, F.Cu at (73.9, 84.1)
- added D35: Green, Diode_SMD:D_0603_1608Metric, F.Cu at (73.9, 81.5)
- added D36: Green, Diode_SMD:D_0603_1608Metric, F.Cu at (82.0, 86.7)
- added D37: Green, Diode_SMD:D_0603_1608Metric, F.Cu at (16.4, 98.4)
- added D38: Green, Diode_SMD:D_0603_1608Metric, F.Cu at (16.7, 85.1)
- added D39: Green, Diode_SMD:D_0603_1608Metric, F.Cu at (90.1, 88.5)
- added D4: Green, Diode_SMD:D_0603_1608Metric, F.Cu at (45.0, 89.7)
- added D40: Green, Diode_SMD:D_0603_1608Metric, F.Cu at (90.1, 83.3)
- added D41: Green, Diode_SMD:D_0603_1608Metric, F.Cu at (94.2, 85.9)
- added D42: Red, Diode_SMD:D_0603_1608Metric, F.Cu at (82.0, 84.1)
- added D43: Green, Diode_SMD:D_0603_1608Metric, F.Cu at (86.0, 86.7)
- added D44: Green, Diode_SMD:D_0603_1608Metric, F.Cu at (20.4, 98.4)
- added D45: Green, Diode_SMD:D_0603_1608Metric, F.Cu at (69.8, 85.9)
- added D46: Green, Diode_SMD:D_0603_1608Metric, F.Cu at (16.7, 82.5)
- added D47: Green, Diode_SMD:D_0603_1608Metric, F.Cu at (82.0, 78.9)
- added D48: Green, Diode_SMD:D_0603_1608Metric, F.Cu at (24.8, 85.0)
- added D49: Green, Diode_SMD:D_0603_1608Metric, F.Cu at (12.4, 105.0)
- added D5: Green, Diode_SMD:D_0603_1608Metric, F.Cu at (16.1, 88.8)
- added D50: Green, Diode_SMD:D_0603_1608Metric, F.Cu at (16.1, 91.3)
- added D51: Green, Diode_SMD:D_0603_1608Metric, F.Cu at (16.4, 101.0)
- added D52: Green, Diode_SMD:D_0603_1608Metric, F.Cu at (78.0, 84.1)
- added D53: Green, Diode_SMD:D_0603_1608Metric, F.Cu at (73.9, 78.9)
- added D54: Green, Diode_SMD:D_0603_1608Metric, F.Cu at (49.4, 93.9)
- added D55: Green, Diode_SMD:D_0603_1608Metric, F.Cu at (25.1, 95.5)
- added D56: Green, Diode_SMD:D_0603_1608Metric, F.Cu at (69.8, 79.9)
- added D57: Green, Diode_SMD:D_0603_1608Metric, F.Cu at (33.2, 93.9)
- added D58: Green, Diode_SMD:D_0603_1608Metric, F.Cu at (20.1, 90.2)
- added D59: Green, Diode_SMD:D_0603_1608Metric, F.Cu at (-6.90, 46.8)
- added D6: Green, Diode_SMD:D_0603_1608Metric, F.Cu at (86.0, 78.9)
- added D60: Green, Diode_SMD:D_0603_1608Metric, F.Cu at (20.8, 87.6)
- added D61: Green, Diode_SMD:D_0603_1608Metric, F.Cu at (79.5, 76.3)
- added D62: Green, Diode_SMD:D_0603_1608Metric, F.Cu at (86.0, 81.5)
- added D63: Green, Diode_SMD:D_0603_1608Metric, F.Cu at (37.0, 89.7)
- added D64: Green, Diode_SMD:D_0603_1608Metric, F.Cu at (76.8, 89.3)
- added D65: Green, Diode_SMD:D_0603_1608Metric, F.Cu at (80.8, 89.3)
- added D66: Green, Diode_SMD:D_0603_1608Metric, F.Cu at (90.1, 80.7)
- added D67: Green, Diode_SMD:D_0603_1608Metric, F.Cu at (78.0, 81.5)
- added D68: Green, Diode_SMD:D_0603_1608Metric, F.Cu at (32.9, 89.7)
- added D69: Blue, Diode_SMD:D_0603_1608Metric, F.Cu at (83.5, 76.3)
- added D7: Green, Diode_SMD:D_0603_1608Metric, F.Cu at (75.5, 76.3)
- added D8: Green, Diode_SMD:D_0603_1608Metric, F.Cu at (20.4, 101.0)
- added D9: Green, Diode_SMD:D_0603_1608Metric, F.Cu at (71.4, 76.3)
- added JP3: SolderJumper_3_Open, Jumper:SolderJumper-3_P1.3mm_Open_RoundedPad1.0x1.5mm, F.Cu at (-51.2, 51.6)
- added R10: 620R, Resistor_SMD:R_0603_1608Metric, F.Cu at (-42.1, 74.3)
- added R11: 2k2, Resistor_SMD:R_0603_1608Metric, F.Cu at (-38.1, 79.3)
- added R12: 2k2, Resistor_SMD:R_0603_1608Metric, F.Cu at (-62.1, 81.8)
- added R13: 20k, Resistor_SMD:R_0603_1608Metric, F.Cu at (-54.2, 76.8)
- added R14: 20k, Resistor_SMD:R_0603_1608Metric, F.Cu at (-58.2, 76.8)
- added R8: 330R, Resistor_SMD:R_0603_1608Metric, F.Cu at (-42.2, 76.8)
- added R9: 80R, Resistor_SMD:R_0603_1608Metric, F.Cu at (-58.1, 79.3)
- added U3: CAT24C256, Package_SO:SOIC-8_3.9x4.9mm_P1.27mm, F.Cu at (-49.9, 57.5)
- added U4: IS31FL3731-QF, Package_DFN_QFN:QFN-28-1EP_4x4mm_P0.4mm_EP2.3x2.3mm, F.Cu at (-62.0, 61.3)
- BT1: moved to F.Cu
- C1: value 100n -> 47pF; footprint Capacitor_SMD:C_0805_2012Metric_Pad1.18x1.45mm_HandSolder -> Capacitor_SMD:C_0603_1608Metric; moved to F.Cu
- C2: value 1uF -> 10uF; footprint Capacitor_SMD:C_0805_2012Metric_Pad1.18x1.45mm_HandSolder -> Capacitor_SMD:C_0603_1608Metric; moved to F.Cu
- C3: value 22pF -> 1uF; footprint Capacitor_SMD:C_0805_2012Metric_Pad1.18x1.45mm_HandSolder -> Capacitor_SMD:C_0603_1608Metric; moved to F.Cu
- D1: value SML522BUNWT86 -> Green; footprint LED_SMD_Rohm:SML522BUNWT86 -> Diode_SMD:D_0603_1608Metric; moved to F.Cu
- D2: value 0.5A 40V 420mV -> Green; footprint Capacitor_SMD:C_0805_2012Metric_Pad1.18x1.45mm_HandSolder -> Diode_SMD:D_0603_1608Metric; moved to F.Cu
- J1: value SSW-120-22-G-D-RA -> ANT_SMA; footprint Connector_Header_Samtec:SAMTEC_SSW-120-22-G-D-RA -> Connector_SMA_Samtec:SAMTEC_SMA-J-P-H-ST-EM1; moved to F.Cu
- J2: value SMA jack -> SSQ-120-03_GPIO; footprint Connector_SMA_Samtec:SAMTEC_SMA-J-P-H-ST-EM1 -> Connector_Header_Samtec:SAMTEC_SSQ-120-03-G-D_Pi; moved to F.Cu
- J3: value TSW-120-08-G-D-RA -> TSM-103-01-L-SV; footprint Connector_Header_Samtec:SAMTEC_TSW-120-08-G-D-RA -> Connector_PinHeader_2.54mm:PinHeader_1x02_P2.54mm_Vertical_SMD_Pin1Right; moved to F.Cu
- JP1: value ID_WP -> TSM-103-01-L-SV; footprint Jumper:SolderJumper-2_P1.3mm_Open_RoundedPad1.0x1.5mm -> Connector_PinHeader_2.54mm:PinHeader_1x02_P2.54mm_Vertical_SMD_Pin1Right; moved to F.Cu
- JP2: value SolderJumper_3_Open -> ID_WP; footprint Jumper:SolderJumper-3_P1.3mm_Open_RoundedPad1.0x1.5mm -> Jumper:SolderJumper-2_P1.3mm_Open_RoundedPad1.0x1.5mm; moved to F.Cu
- L1: value LQG15HS33NJ02D -> 47nH; footprint Inductor_SMD_Murata:INDC1005X55N -> Inductor_SMD:L_0603_1608Metric; moved to F.Cu
- R1: value 3.9k -> 10R; footprint Resistor_SMD:R_0805_2012Metric_Pad1.20x1.40mm_HandSolder -> Resistor_SMD:R_0603_1608Metric; moved to F.Cu
- R2: value 3.9k -> DNP; moved to F.Cu
- R3: value 620R -> 20k; footprint Resistor_SMD:R_0805_2012Metric_Pad1.20x1.40mm_HandSolder -> Resistor_SMD:R_0603_1608Metric; moved to F.Cu
- R4, R5: value 2k2 -> 20k; footprint Resistor_SMD:R_0805_2012Metric_Pad1.20x1.40mm_HandSolder -> Resistor_SMD:R_0603_1608Metric; moved to F.Cu
- R6: value 280R -> 3.9k; footprint Resistor_SMD:R_0805_2012Metric_Pad1.20x1.40mm_HandSolder -> Resistor_SMD:R_0603_1608Metric; moved to F.Cu
- R7: value 80R -> 3.9k; footprint Resistor_SMD:R_0805_2012Metric_Pad1.20x1.40mm_HandSolder -> Resistor_SMD:R_0603_1608Metric; moved to F.Cu
- U1: value CAT24C256 -> MAX-M10S; footprint Package_SO:SOIC-8_3.9x4.9mm_P1.27mm -> RF_GNSS_u-blox:MAX-M10S; moved to F.Cu
- U2: value MAX-M10S -> PCA9557PW; footprint RF_GNSS_u-blox:MAX-M10S -> Package_SO:TSSOP-16_4.4x5mm_P0.65mm; moved to F.Cu
- moved U2 225.4 mm to (-71.9, 68.6)
- moved L1 212.9 mm to (-58.1, 81.8)
- moved JP1 210.1 mm to (-72.3, 75.5), turned to 0 degrees
- moved R1 199.1 mm to (-54.1, 79.3), turned to 0 degrees
- moved BT1 199.0 mm to (-61.0, 54.0)
- moved J3 197.7 mm to (-63.5, 68.9)
- moved C3 197.7 mm to (-42.1, 79.3), turned to 0 degrees
- moved C2 197.6 mm to (-54.1, 81.8), turned to 0 degrees
- moved J1 190.5 mm to (-70.7, 53.1)
- moved C1 179.9 mm to (-37.5, 71.8), turned to 0 degrees
- moved JP2 177.7 mm to (-46.2, 51.6), turned to 0 degrees
- moved R5 175.7 mm to (-46.2, 76.8), turned to 0 degrees
- moved R4 170.1 mm to (-46.1, 79.3), turned to 0 degrees
- moved R6 167.9 mm to (-45.5, 71.8), turned to 0 degrees
- moved U1 165.8 mm to (-15.7, 48.4), turned to 0 degrees
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Connections:
- C1 pad 1: +3V3 -> Net-(C1-Pad1)
- C1 pad 2: GND -> /GNSS_RF_IN
- C2 pad 1: /GNSS_VBCKP -> +3V3
- C3 pad 1: GND -> +3V3
- C3 pad 2: +3V3 -> GND
- D1 pad 1: Net-(R6-Pad2) -> /CA1
- D1 pad 2: GND -> /CA2
- D2 pad 1: Net-(D2-Pad1) -> /CA1
- D2 pad 2: +3V3 -> Net-(D10-Pad2)
- JP1 pad 1: /WP -> Net-(C1-Pad1)
- JP1 pad 2: +3V3 -> Net-(JP1-Pad2)
- JP2 pad 1: Net-(JP2-Pad1) -> /WP
- L1 pad 1: +3V3 -> Net-(JP1-Pad2)
- L1 pad 2: /GNSS_RF_IN -> Net-(L1-Pad2)
- R1 pad 1: +3V3 -> Net-(L1-Pad2)
- R1 pad 2: /ID_SDA -> Net-(R1-Pad2)
- R2 pad 1: +3V3 -> /GPIO[5]
- R2 pad 2: /ID_SCL -> +3V3
- R3 pad 1: Net-(D2-Pad1) -> GND
- R3 pad 2: /GNSS_VBCKP -> Net-(R3-Pad2)
- R4 pad 1: Net-(JP2-Pad3) -> GND
- R4 pad 2: /GNSS_SDA -> Net-(R4-Pad2)
- R5 pad 1: Net-(JP2-Pad1) -> GND
- R5 pad 2: /GNSS_SCL -> Net-(R5-Pad2)
- R6 pad 2: Net-(R6-Pad2) -> /ID_SDA
- R7 pad 1: /GNSS_PPS -> +3V3
- R7 pad 2: Net-(R7-Pad2) -> /ID_SCL
- U1 pad 1: unconnected-(U1-Pad1) -> GND
- U1 pad 2: unconnected-(U1-Pad2) -> /GNSS_TX
- U1 pad 3: unconnected-(U1-Pad3) -> /GNSS_RX
- U1 pad 4: GND -> /GNSS_PPS
- U1 pad 5: /ID_SDA -> unconnected-(U1-Pad5)
- U1 pad 6: /ID_SCL -> /GNSS_VBCKP
- U1 pad 7: /WP -> +3V3
- U2 pad 1: GND -> /GNSS_SCL
- U2 pad 10: GND -> /~{LEDMATRIX_INT}
- U2 pad 11: /GNSS_RF_IN -> unconnected-(U2-Pad11)
- U2 pad 12: GND -> unconnected-(U2-Pad12)
- U2 pad 13: /GNSS_LNA_EN -> unconnected-(U2-Pad13)
- U2 pad 15: unconnected-(U2-Pad15) -> /GPIO[5]
- U2 pad 16: /GNSS_SDA -> +3V3
- U2 pad 2: /GNSS_TX -> /GNSS_SDA
- U2 pad 3: /GNSS_RX -> Net-(R3-Pad2)
- U2 pad 4: /GNSS_PPS -> Net-(R4-Pad2)
- U2 pad 5: unconnected-(U2-Pad5) -> Net-(R5-Pad2)
- U2 pad 6: /GNSS_VBCKP -> /~{GNSS_RESET}
- U2 pad 7: +3V3 -> /~{GNSS_SAFEBOOT}
- U2 pad 8: +3V3 -> GND
- U2 pad 9: unconnected-(U2-Pad9) -> /~{LEDMATRIX_OFF}
Routing:
- net GND: track 609.9 -> 0.00 mm, vias 70 -> 0
- net +3V3: track 209.3 -> 0.00 mm, vias 3 -> 0
- net /GNSS_SDA: track 133.2 -> 0.00 mm, vias 1 -> 0
- net /GNSS_SCL: track 130.5 -> 0.00 mm, vias 1 -> 0
- net /GNSS_RX: track 107.0 -> 0.00 mm, vias 1 -> 0
- net /GNSS_TX: track 104.0 -> 0.00 mm, vias 1 -> 0
- net /GNSS_PPS: track 101.1 -> 0.00 mm, vias 1 -> 0
- net /ID_SDA: track 81.4 -> 0.00 mm, vias 1 -> 0
- net /GPIO[4]/GPCLK0: track 76.7 -> 0.00 mm
- net +5V: track 76.1 -> 0.00 mm
- net /GPIO[17]: track 75.9 -> 0.00 mm
- net /GPIO[27]: track 75.4 -> 0.00 mm
- net /GPIO[22]: track 75.0 -> 0.00 mm
- net /GPIO[9]/SPI0.MISO: track 74.2 -> 0.00 mm
- net /GPIO[10]/SPI0.MOSI: track 74.1 -> 0.00 mm
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- removed copper zone on B.Cu, net GND
- removed copper zone on F.Cu, net GND
Other:
- board size 65 x 76 mm -> 65 x 56 mm
- board text added: "PoE"
- board text removed: "JLCJLCJLCJLC"
- board text removed: "red: +3V3 blue: pps"

Commit message: rev2 prep
Parts:
- moved J1 190.4 mm to (119.7, 55.3), turned to 90 degrees
- moved C1 154.0 mm to (115.7, 55.3), turned to 180 degrees
- moved U1 123.5 mm to (107.8, 52.0)
- moved U4 119.4 mm to (51.0, 99.8)
- moved D59 109.5 mm to (93.9, 89.7)
- moved D3 74.1 mm to (74.3, 71.1), turned to -90 degrees
- moved D8 70.1 mm to (83.8, 71.1), turned to -90 degrees
- moved D5 64.5 mm to (78.1, 71.1), turned to -90 degrees
- moved D11 52.1 mm to (75.4, 109.1)
- moved D12 52.1 mm to (92.2, 104.6)
- moved D13 52.1 mm to (67.5, 116.9)
- moved D16 52.1 mm to (92.0, 100.4)
- moved D23 52.1 mm to (71.7, 95.7)
- moved D24 52.1 mm to (67.5, 114.3)
- moved D27 52.1 mm to (88.2, 104.6)
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Routing:
- added copper zone on F.Cu, net (none)

Commit message: rev2 prep
Parts:
- added D70: Green, Diode_SMD:D_0603_1608Metric, F.Cu at (92.7, 109.9)
- added D71: Green, Diode_SMD:D_0603_1608Metric, F.Cu at (88.7, 109.9)
- added D72: Green, Diode_SMD:D_0603_1608Metric, F.Cu at (96.8, 109.9)
- added D73: Green, Diode_SMD:D_0603_1608Metric, F.Cu at (88.7, 112.4)
- added D74: Green, Diode_SMD:D_0603_1608Metric, F.Cu at (92.7, 112.4)
- added D75: Green, Diode_SMD:D_0603_1608Metric, F.Cu at (96.8, 112.4)
- moved D61 59.3 mm to (134.0, 99.7), turned to -90 degrees
- moved D69 45.9 mm to (128.3, 66.0)
- moved D42 44.3 mm to (121.9, 64.8)
- moved D14 42.9 mm to (141.0, 76.8)
- moved D21 39.9 mm to (134.0, 81.9)
- moved D62 37.1 mm to (118.7, 99.1)
- moved D29 35.8 mm to (129.5, 86.4)
- moved D32 27.9 mm to (59.7, 76.8)
- moved D47 23.8 mm to (104.8, 85.7)
- moved D67 17.3 mm to (94.0, 74.9)
Connections:
- D10 pad 2: Net-(D10-Pad2) -> /CA3
- D11 pad 2: Net-(D11-Pad2) -> /CA4
- D12 pad 2: Net-(D12-Pad2) -> /CA5
- D13 pad 2: Net-(D13-Pad2) -> /CA6
- D14 pad 2: Net-(D14-Pad2) -> /CA7
- D15 pad 2: Net-(D15-Pad2) -> /CA8
- D19 pad 2: Net-(D11-Pad2) -> /CA4
- D2 pad 2: Net-(D10-Pad2) -> /CA3
- D20 pad 2: Net-(D12-Pad2) -> /CA5
- D21 pad 2: Net-(D13-Pad2) -> /CA6
- D22 pad 2: Net-(D14-Pad2) -> /CA7
- D23 pad 2: Net-(D15-Pad2) -> /CA8
- D28 pad 2: Net-(D10-Pad2) -> /CA3
- D29 pad 2: Net-(D12-Pad2) -> /CA5
- D3 pad 2: Net-(D11-Pad2) -> /CA4
- D30 pad 2: Net-(D13-Pad2) -> /CA6
- D31 pad 2: Net-(D14-Pad2) -> /CA7
- D32 pad 2: Net-(D15-Pad2) -> /CA8
- D36 pad 2: Net-(D10-Pad2) -> /CA3
- D37 pad 2: Net-(D11-Pad2) -> /CA4
- D38 pad 2: Net-(D13-Pad2) -> /CA6
- D39 pad 2: Net-(D14-Pad2) -> /CA7
- D4 pad 2: Net-(D12-Pad2) -> /CA5
- D40 pad 2: Net-(D15-Pad2) -> /CA8
- D45 pad 2: Net-(D10-Pad2) -> /CA3
- D46 pad 2: Net-(D11-Pad2) -> /CA4
- D47 pad 2: Net-(D12-Pad2) -> /CA5
- D48 pad 2: Net-(D14-Pad2) -> /CA7
- D49 pad 2: Net-(D15-Pad2) -> /CA8
- D5 pad 2: Net-(D13-Pad2) -> /CA6
- D53 pad 2: Net-(D10-Pad2) -> /CA3
- D54 pad 2: Net-(D11-Pad2) -> /CA4
- D55 pad 2: Net-(D12-Pad2) -> /CA5
- D56 pad 2: Net-(D13-Pad2) -> /CA6
- D57 pad 2: Net-(D15-Pad2) -> /CA8
- D6 pad 2: Net-(D14-Pad2) -> /CA7
- D61 pad 2: Net-(D10-Pad2) -> /CA3
- D62 pad 2: Net-(D11-Pad2) -> /CA4
- D63 pad 2: Net-(D12-Pad2) -> /CA5
- D64 pad 2: Net-(D13-Pad2) -> /CA6
- D65 pad 2: Net-(D14-Pad2) -> /CA7
- D7 pad 2: Net-(D15-Pad2) -> /CA8

Commit message: rev2 prep
Parts:
- removed C10, C11: 10uF, Capacitor_SMD:C_0603_1608Metric
- removed C12: 1uF, Capacitor_SMD:C_0603_1608Metric
- removed C13: 0.1uF, Capacitor_SMD:C_0603_1608Metric
- removed D1, D10, D11, D12, D13, D14, D15, D16, D17, D18, D19, D2, D20, D21, D22, D23, D24, D26, D27, D28, D29, D3, D30, D31, D32, D33, D34, D35, D36, D37, D38, D39, D4, D40, D41, D43, D44, D45, D46, D47, D48, D49, D5, D50, D51, D52, D53, D54, D55, D56, D57, D58, D59, D6, D60, D61, D62, D63, D64, D65, D66, D67, D68, D7, D70, D71, D72, D73, D74, D75, D8, D9: Green, Diode_SMD:D_0603_1608Metric
- removed R13, R14: 20k, Resistor_SMD:R_0603_1608Metric
- removed U4: IS31FL3731-QF, Package_DFN_QFN:QFN-28-1EP_4x4mm_P0.4mm_EP2.3x2.3mm
- moved D25 54.1 mm to (141.6, 69.2), turned to -90 degrees
