File: picise.kicad_pcb (KiCad board)
At the start: 2 copper layers, 65 x 56 mm, 41 parts, among them J1 ANT_SMA, J2 SSQ-120-03_GPIO, J3 TSM-103-01-L-SV, U1 MAX-M10S, U2 PCA9557PW, U3 CAT24C256

Commit message: rev2 prep
Parts:
- moved BT1 151.1 mm to (90.1, 55.2)
- moved U3 142.9 mm to (92.7, 48.3)
- moved D69 40.9 mm to (87.6, 61.6)
- moved D25 34.2 mm to (108.0, 62.9), turned to 0 degrees
- moved D42 26.9 mm to (95.2, 61.6)
- moved U1 1.33 mm to (107.8, 50.7)
- moved C1 1.32 mm to (115.7, 54.0)
- moved J1 1.32 mm to (119.7, 54.0)
Other:
- board text removed: "PoE"
Changed lines of the file:
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@@
   )
   (footprint "Capacitor_SMD:C_0603_1608Metric" (layer "F.Cu")
-    (at 115.65 55.3 180)
+    (at 115.65 53.975 180)
     (descr "Capacitor SMD 0603 (1608 Metric), square (rectangular) end terminal, IPC_7351 nominal, (Body size source: IPC-SM-782 page 76, https://www.pcb-3d.com/wordpress/wp-content/uploads/ipc-sm-782a_amendment_1_and_2.pdf), generated with kicad-footprint-generator")
     (tags "capacitor")
@@
     (property "Sheetname" "")
     (attr smd)
-    (fp_text reference "C1" (at 0 -1.43) (layer "F.SilkS")
-      (effects (font (size 1 1) (thickness 0.15)))
-    )
-    (fp_text value "47pF" (at 0 1.43) (layer "F.Fab")
-      (effects (font (size 1 1) (thickness 0.15)))
+    (fp_text reference "C1" (at 0 -1.43) (layer "F.SilkS") hide
+      (effects (font (size 1 1) (thickness 0.15)))
+    )
+    (fp_text value "47pF" (at 0 1.27) (layer "F.Fab")
+      (effects (font (size 0.3 0.3) (thickness 0.075)))
     )
     (fp_text user "${REFERENCE}" (at 0 0) (layer "F.Fab")
@@
   )
   (footprint "Connector_SMA_Samtec:SAMTEC_SMA-J-P-H-ST-EM1" (layer "F.Cu")
-    (at 119.7 55.3 90)
+    (at 119.7 53.975 90)
     (descr "SMA Connector Jack, Female Socket 50Ohm Board Edge, End Launch Solder")
     (property "Digikey" "SMA-J-P-H-ST-EM1")
@@
     (property "Sheetname" "")
     (attr through_hole)
-    (fp_text reference "J1" (at -0.34105 -3.66967 90) (layer "F.SilkS")
-      (effects (font (size 1 1) (thickness 0.15)))
-    )
-    (fp_text value "ANT_SMA" (at 0 12.6 90) (layer "F.Fab")
-      (effects (font (size 1 1) (thickness 0.15)))
-    )
-    (fp_text user "PCB EDGE" (at 5.8 1.4 90) (layer "F.Fab")
-      (effects (font (size 0.48 0.48) (thickness 0.15)))
+    (fp_text reference "J1" (at -2.54 -3.495 90) (layer "F.SilkS") hide
+      (effects (font (size 1 1) (thickness 0.15)))
+    )
+    (fp_text value "ANT_SMA" (at 1.27 0.315 180) (layer "F.Fab")
+      (effects (font (size 0.3 0.3) (thickness 0.075)))
     )
     (fp_line (start -1.8 -1.91) (end -1 -1.91) (layer "F.SilkS") (width 0.2))
@@
   )
   (footprint "Battery_Cell_Seiko:BAT_MS621FE-FL11E" (layer "F.Cu")
-    (at -61 54)
+    (at 90.065 55.245)
     (property "Digikey" "MS621FE-FL11E")
     (property "MPN" "MS621FE-FL11E")
@@
       (effects (font (size 1 1) (thickness 0.15)))
     )
-    (fp_text value "MS621FE-FL11E" (at 6.985 4.445) (layer "F.Fab")
-      (effects (font (size 1 1) (thickness 0.15)))
+    (fp_text value "MS621FE-FL11E" (at 0 0) (layer "F.Fab")
+      (effects (font (size 0.3 0.3) (thickness 0.075)))
     )
     (fp_line (start 5.1 -1.846) (end 5.1 -1.446) (layer "F.SilkS") (width 0.127))
@@
   )
   (footprint "Diode_SMD:D_0603_1608Metric" (layer "F.Cu")
-    (at 141.605 69.215 -90)
+    (at 107.95 62.865)
     (descr "Diode SMD 0603 (1608 Metric), square (rectangular) end terminal, IPC_7351 nominal, (Body size source: http://www.tortai-tech.com/upload/download/2011102023233369053.pdf), generated with kicad-footprint-generator")
     (tags "diode")
@@
     (property "Sheetname" "")
     (attr smd)
-    (fp_text reference "D25" (at 0 -1.43 90) (layer "F.SilkS")
-      (effects (font (size 1 1) (thickness 0.15)))
-    )
-    (fp_text value "0.5A 40V 420mV" (at 0 1.43 90) (layer "F.Fab")
-      (effects (font (size 1 1) (thickness 0.15)))
-    )
-    (fp_text user "${REFERENCE}" (at 0 0 90) (layer "F.Fab")
+    (fp_text reference "D25" (at 0 -1.43) (layer "F.SilkS") hide
+      (effects (font (size 1 1) (thickness 0.15)))
+    )
+    (fp_text value "0.5A 40V 420mV" (at 0 1.27) (layer "F.Fab")
+      (effects (font (size 0.3 0.3) (thickness 0.075)))
+    )
+    (fp_text user "${REFERENCE}" (at 0 0) (layer "F.Fab")
       (effects (font (size 0.4 0.4) (thickness 0.06)))
     )
@@
     (fp_line (start -0.5 -0.4) (end -0.8 -0.1) (layer "F.Fab") (width 0.1))
     (fp_line (start -0.8 0.4) (end 0.8 0.4) (layer "F.Fab") (width 0.1))
-    (pad "1" smd roundrect (at -0.7875 0 270) (size 0.875 0.95) (layers "F.Cu" "F.Paste" "F.Mask") (roundrect_rratio 0.25)
+    (pad "1" smd roundrect (at -0.7875 0) (size 0.875 0.95) (layers "F.Cu" "F.Paste" "F.Mask") (roundrect_rratio 0.25)
       (net 6 "Net-(D25-Pad1)") (pinfunction "K") (pintype "passive"))
-    (pad "2" smd roundrect (at 0.7875 0 270) (size 0.875 0.95) (layers "F.Cu" "F.Paste" "F.Mask") (roundrect_rratio 0.25)
+    (pad "2" smd roundrect (at 0.7875 0) (size 0.875 0.95) (layers "F.Cu" "F.Paste" "F.Mask") (roundrect_rratio 0.25)
       (net 5 "+3V3") (pinfunction "A") (pintype "passive"))
     (model "${KICAD6_3DMODEL_DIR}/Diode_SMD.3dshapes/D_0603_1608Metric.wrl"
@@
   )
   (footprint "Diode_SMD:D_0603_1608Metric" (layer "F.Cu")
-    (at 121.92 64.77)
+    (at 95.25 61.595)
     (descr "Diode SMD 0603 (1608 Metric), square (rectangular) end terminal, IPC_7351 nominal, (Body size source: http://www.tortai-tech.com/upload/download/2011102023233369053.pdf), generated with kicad-footprint-generator")
     (tags "diode")
@@
     (property "Sheetname" "")
     (attr smd)
-    (fp_text reference "D42" (at 0 -1.43) (layer "F.SilkS")
-      (effects (font (size 1 1) (thickness 0.15)))
-    )
-    (fp_text value "Red" (at 0 1.43) (layer "F.Fab")
-      (effects (font (size 1 1) (thickness 0.15)))
+    (fp_text reference "D42" (at 0 -1.43) (layer "F.SilkS") hide
+      (effects (font (size 1 1) (thickness 0.15)))
+    )
+    (fp_text value "Red" (at 0 1.27) (layer "F.Fab")
+      (effects (font (size 0.3 0.3) (thickness 0.075)))
     )
     (fp_text user "${REFERENCE}" (at 0 0) (layer "F.Fab")
@@
   )
   (footprint "Package_SO:SOIC-8_3.9x4.9mm_P1.27mm" (layer "F.Cu")
-    (at -49.85 57.47)
+    (at 92.71 48.26)
     (descr "SOIC, 8 Pin (JEDEC MS-012AA, https://www.analog.com/media/en/package-pcb-resources/package/pkg_pdf/soic_narrow-r/r_8.pdf), generated with kicad-footprint-generator ipc_gullwing_generator.py")
     (tags "SOIC SO")
@@
   )
   (footprint "RF_GNSS_u-blox:MAX-M10S" (layer "F.Cu")
-    (at 107.75 52)
+    (at 107.75 50.675)
     (descr "Standard precision GNSS module, ultra-low-power")
     (property "MPN" "MAX-M10S-00B")
@@
     )
     (fp_text value "MAX-M10S" (at -0.055 0.7 unlocked) (layer "F.Fab")
-      (effects (font (size 0.5 0.5) (thickness 0.1)))
+      (effects (font (size 0.3 0.3) (thickness 0.075)))
     )
     (fp_text user "${REFERENCE}" (at 0 -0.38) (layer "F.Fab")
@@
   )
   (footprint "Diode_SMD:D_0603_1608Metric" (layer "F.Cu")
-    (at 128.27 66.04)
+    (at 87.63 61.595)
     (descr "Diode SMD 0603 (1608 Metric), square (rectangular) end terminal, IPC_7351 nominal, (Body size source: http://www.tortai-tech.com/upload/download/2011102023233369053.pdf), generated with kicad-footprint-generator")
     (tags "diode")
@@
     (property "Sheetname" "")
     (attr smd)
-    (fp_text reference "D69" (at 0 -1.43) (layer "F.SilkS")
-      (effects (font (size 1 1) (thickness 0.15)))
-    )
-    (fp_text value "Blue" (at 0 1.43) (layer "F.Fab")
-      (effects (font (size 1 1) (thickness 0.15)))
+    (fp_text reference "D69" (at 0 -1.43) (layer "F.SilkS") hide
+      (effects (font (size 1 1) (thickness 0.15)))
+    )
+    (fp_text value "Blue" (at 0 1.27) (layer "F.Fab")
+      (effects (font (size 0.3 0.3) (thickness 0.075)))
     )
     (fp_text user "${REFERENCE}" (at 0 0) (layer "F.Fab")
@@
   (gr_line (start 59.63 94.23) (end 118.63 94.23) (layer "Edge.Cuts") (width 0.1))
   (gr_arc (start 118.63 38.23) (mid 120.75132 39.10868) (end 121.63 41.23) (layer "Edge.Cuts") (width 0.1))
-  (gr_text "PoE" (at 118.13 47.87) (layer "Dwgs.User")
-    (effects (font (size 1 1) (thickness 0.15)))
-  )
   (zone (net 0) (net_name "") (layer "F.Cu") (hatch edge 0.508)
     (connect_pads (clearance 0))
@@
       )
     )
-  )
-  (zone (net 0) (net_name "") (layer "B.Cu") (name "PoE") (hatch full 0.508)
-    (connect_pads (clearance 0))
-    (min_thickness 0.254)
-    (keepout (tracks allowed) (vias allowed) (pads allowed) (copperpour allowed) (footprints not_allowed))
-    (fill (thermal_gap 0.508) (thermal_bridge_width 0.508))
-    (polygon
-      (pts
-        (xy 120.63 50.37)
-        (xy 115.63 50.37)
-        (xy 115.63 45.37)
-        (xy 120.63 45.37)
-      )
-    )

Commit message: rev2 prep
Parts:
- moved U2 166.5 mm to (93.3, 48.3)
- moved U3 15.2 mm to (77.5, 48.3)

Commit message: rev2 prep
Parts:
- added DS1: NHD-C12832A1Z-FSW-FBW-3V3, Display_LCD_Newhaven:LCD_NHD-C12832A1Z-FSW-FBW-3V3, F.Cu at (88.9, 81.3)
- moved U2 17.0 mm to (77.4, 54.2)
- moved BT1 2.86 mm to (91.3, 52.7)
Connections:
- J2 pad 23: /GPIO[11]/SPI0.SCLK -> /DISP_SCLK
- U2 pad 10: /~{LEDMATRIX_INT} -> unconnected-(U2-Pad10)
- U2 pad 9: /~{LEDMATRIX_OFF} -> /~{DISP_RST}
