File: picise.kicad_pcb (KiCad board)
At the start: 2 copper layers, 65 x 56 mm, 42 parts, among them J1 ANT_SMA, J2 SSQ-120-03_GPIO, J3 TSM-103-01-L-SV, U1 MAX-M10S, U2 PCA9557PW, U3 CAT24C256

Commit message: rev2 prep
Parts:
- DS1: value NHD-C12832A1Z-FSW-FBW-3V3 -> NHD-3.12-25664UCB2_SPI; footprint Display_LCD_Newhaven:LCD_NHD-C12832A1Z-FSW-FBW-3V3 -> Display_OLED_Newhaven:OLED_NHD-3.12-25664UCx2
- moved D69 20.1 mm to (88.9, 81.7)
- moved D42 19.1 mm to (88.9, 79.7)
- moved DS1 6.63 mm to (88.9, 87.9)
Connections:
- net /GPIO[8]/SPI0.CE0 renamed /~{DISP_CE0}
- DS1 pad 1: unconnected-(DS1-Pad1) -> GND
- DS1 pad 10: unconnected-(DS1-Pad10) -> GND
- DS1 pad 11: unconnected-(DS1-Pad11) -> GND
- DS1 pad 12: unconnected-(DS1-Pad12) -> GND
- DS1 pad 13: /GPIO[10]/SPI0.MOSI -> GND
- DS1 pad 14: /DISP_SCLK -> GND
- DS1 pad 2: unconnected-(DS1-Pad2) -> +3V3
- DS1 pad 4: unconnected-(DS1-Pad4) -> /DISP_D_C
- DS1 pad 5: unconnected-(DS1-Pad5) -> GND
- DS1 pad 6: unconnected-(DS1-Pad6) -> /DISP_SCLK
- DS1 pad 7: unconnected-(DS1-Pad7) -> /DISP_MOSI
- DS1 pad 9: unconnected-(DS1-Pad9) -> GND
- J2 pad 19: /GPIO[10]/SPI0.MOSI -> /DISP_MOSI
- J2 pad 37: /GPIO[26] -> /DISP_D_C

Commit message: rev2 draft routed
Parts:
- removed J3, JP1: TSM-103-01-L-SV, Connector_PinHeader_2.54mm:PinHeader_1x02_P2.54mm_Vertical_SMD_Pin1Right
- added C10: 10uF, Capacitor_SMD:C_0603_1608Metric, F.Cu at (105.9, 71.7)
- added C11: 10uF, Capacitor_SMD:C_0603_1608Metric, F.Cu at (107.7, 71.7)
- added C12: 1uF, Capacitor_SMD:C_0603_1608Metric, F.Cu at (109.4, 71.7)
- added C13: 0.1uF, Capacitor_SMD:C_0603_1608Metric, F.Cu at (111.2, 71.7)
- moved L1 177.1 mm to (116.1, 49.8), turned to 90 degrees
- moved C15 171.4 mm to (118.6, 49.4), turned to 180 degrees
- moved R1 171.3 mm to (114.6, 49.8), turned to -90 degrees
- moved C4 156.0 mm to (100.7, 55.2), turned to -90 degrees
- moved C2 153.8 mm to (97.4, 55.6), turned to -90 degrees
- moved R9 143.9 mm to (85.8, 81.7)
- moved C3 143.0 mm to (99.1, 56.6), turned to -90 degrees
- moved R10 141.3 mm to (97.4, 52.5), turned to 90 degrees
- moved R12 138.0 mm to (70.9, 45.3), turned to 180 degrees
- moved C14 136.2 mm to (85.4, 53.4), turned to 90 degrees
- moved R8 134.2 mm to (92.0, 79.7), turned to 180 degrees
- moved R4 126.0 mm to (75.7, 46.9), turned to 180 degrees
- moved R5 125.9 mm to (75.7, 45.3), turned to 180 degrees
- moved C9 125.7 mm to (70.9, 54.4), turned to 180 degrees
- moved C6 125.2 mm to (61.2, 57.8), turned to -90 degrees
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Connections:
- net /~{DISP_CE0} renamed /GPIO[8]/SPI0.CE0
- L1 pad 1: Net-(JP1-Pad2) -> Net-(C1-Pad1)
Routing:
- net +3V3: track 0.00 -> 158.1 mm, vias 0 -> 3
- net /GNSS_PPS: track 0.00 -> 102.9 mm, vias 0 -> 4
- net /GNSS_SCL: track 0.00 -> 90.3 mm, vias 0 -> 2
- net /GNSS_SDA: track 0.00 -> 86.1 mm, vias 0 -> 2
- net /GPIO[5]: track 0.00 -> 76.5 mm, vias 0 -> 1
- net /~{GNSS_SAFEBOOT}: track 0.00 -> 64.7 mm
- net /~{GNSS_RESET}: track 0.00 -> 51.6 mm
- net /~{DISP_RST}: track 0.00 -> 46.2 mm, vias 0 -> 2
- net /GPIO[8]/SPI0.CE0: track 0.00 -> 39.1 mm, vias 0 -> 1
- net /ID_SCL: track 0.00 -> 38.3 mm, vias 0 -> 1
- net /GNSS_RX: track 0.00 -> 34.5 mm, vias 0 -> 1
- net GND: track 0.00 -> 32.7 mm, vias 0 -> 54
- net /GNSS_TX: track 0.00 -> 31.5 mm, vias 0 -> 1
- net /ID_SDA: track 0.00 -> 31.3 mm, vias 0 -> 1
- net /DISP_MOSI: track 0.00 -> 29.6 mm
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- added copper zone on B.Cu, net GND
- added copper zone on F.Cu, net GND
- removed copper zone on F.Cu, net (none)
