File: picise.kicad_pcb (KiCad board)
At the start: 2 copper layers, 65 x 56 mm, 44 parts, among them J1 ANT_SMA, J2 SSQ-120-03_GPIO, U1 MAX-M10S, U2 PCA9557PW, U3 CAT24C256

Commit message: tweaks
Parts:
- removed C10, C11: 10uF, Capacitor_SMD:C_0603_1608Metric
- removed C12: 1uF, Capacitor_SMD:C_0603_1608Metric
- removed C13: 0.1uF, Capacitor_SMD:C_0603_1608Metric
- removed DS1: NHD-3.12-25664UCB2_SPI, Display_OLED_Newhaven:OLED_NHD-3.12-25664UCx2
- removed MH3, MH4: MountingHole_2.7mm_M2.5, MountingHole:MountingHole_2.7mm_M2.5
- added REF**: OSHW-Logo2_14.6x12mm_SilkScreen, Symbol:OSHW-Logo2_14.6x12mm_SilkScreen, B.Cu at (75.5, 56.0)
- moved R9 45.5 mm to (115.4, 47.2)
- moved D69 45.4 mm to (118.4, 47.2)
- moved D42 45.0 mm to (118.4, 45.7), turned to 180 degrees
- moved R8 41.3 mm to (115.4, 45.7), turned to 0 degrees
- moved BT1 3.86 mm to (91.4, 48.8), turned to -90 degrees
- moved C14 1.49 mm to (86.9, 53.8), turned to -90 degrees
- moved C3 0.96 mm to (98.4, 55.9)
- moved C2 0.96 mm to (96.7, 55.0)
- moved C4 0.96 mm to (100.0, 54.6)
- moved D25 0.96 mm to (98.4, 52.9)
- moved R10 0.96 mm to (96.7, 51.9)
- moved R2 0.25 mm to (58.9, 54.4), turned to -90 degrees
- moved C15 0.20 mm to (118.4, 49.4)
Connections:
- J2 pad 19: /DISP_MOSI -> /GPIO[10]/SPI0.MOSI
- J2 pad 23: /DISP_SCLK -> /GPIO[11]/SPI0.SCLK
- J2 pad 37: /DISP_D_C -> /GPIO[26]
- U2 pad 9: /~{DISP_RST} -> unconnected-(U2-Pad9)
Routing:
- net /GNSS_PPS: track 102.9 -> 45.4 mm, vias 4 -> 3
- net +3V3: track 158.1 -> 110.1 mm, vias 3 -> 1
- net /~{DISP_RST}: track 46.2 -> 0.00 mm, vias 2 -> 0
- net /GPIO[8]/SPI0.CE0: track 39.1 -> 0.00 mm, vias 1 -> 0
- net /DISP_MOSI: track 29.6 -> 0.00 mm
- net /DISP_SCLK: track 29.4 -> 0.00 mm
- net /DISP_D_C: track 29.2 -> 0.00 mm
- net /GPIO[5]: track 76.5 -> 60.7 mm, vias 1 -> 2
- net /GNSS_SCL: track 90.3 -> 82.2 mm, vias 2 -> 1
- net /~{GNSS_SAFEBOOT}: track 64.7 -> 59.2 mm
- net /ID_SDA: track 31.3 -> 36.7 mm
- net /GNSS_SDA: track 86.1 -> 81.9 mm, vias 2 -> 1
- net /ID_SCL: track 38.3 -> 34.5 mm
- net /~{GNSS_RESET}: track 51.6 -> 48.6 mm
- net Net-(R4-Pad2): track 20.1 -> 22.2 mm
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Other:
- board size 65 x 56 mm -> 65 x 23.5 mm
- board text added: "+"
- board text added: "I2C PU"
- board text added: "P"
- board text added: "Picise - Raspberry Pi GNSS"
- board text added: "WP"

Commit message: more rev2 work
Routing:
- net /~{GNSS_RESET}: track 48.6 -> 47.8 mm
- net /ID_SCL: track 34.5 -> 33.8 mm

Commit message: updated renders
Parts:
- added ?: LOGO, Graphics:by-sa 15x5.2, B.Cu at (78.0, 53.0)
- moved REF** 24.1 mm to (99.3, 53.0)
Other:
- board text added: "Copyright (C) 2022 Christian Kuhtz"
- board text added: "https://github.com/ckuhtz/picise"
- board text added: "rev2"
